File: ngspice_filtro_pasivo.kicad_pcb (KiCad board)
At the start: 2 copper layers, 90 x 60 mm, 8 parts

Commit message: agregando documentos de fabricacion
Other:
- board text added: "0,0000 mm / 0,0000 mm"
- board text added: "0,3000 mm"
- board text added: "1,6000 mm"
- board text added: "2"
- board text added: "90,0000 mm x 60,0000 mm"
- board text added: "Bordes de la placa revestidos:"
- board text added: "CARACTERÍSTICAS DE LA PLACA"
- board text added: "Conectores laterales de tarjeta:"
- board text added: "Control de impedancia:"
- board text added: "Dimensiones generales de la placa:"
- board text added: "Diámetro mínimo de orificio:"
- board text added: "Grosor de la placa:"
- board text added: "No"
- board text added: "None"
- board text added: "Número de capas de cobre:"
- board text added: "Pads castellados:"
- board text added: "Pista/espaciado mínimo:"
- board text added: "Terminación de cobre:"
Changed lines of the file:
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@@
     (effects (font (size 2 2) (thickness 0.2)) (justify left bottom))
   )
-  (dimension (type aligned) (layer "Edge.Cuts")
+  (gr_text "Diámetro mínimo de orificio: " (at 91.721423 24.75) (layer "Cmts.User")
+    (effects (font (size 1.5 1.5) (thickness 0.2)) (justify left top))
+  )
+  (gr_text "Control de impedancia: " (at 91.721423 28.25) (layer "Cmts.User")
+    (effects (font (size 1.5 1.5) (thickness 0.2)) (justify left top))
+  )
+  (gr_text "" (at 129.778565 21.25) (layer "Cmts.User")
+    (effects (font (size 1.5 1.5) (thickness 0.2)) (justify left top))
+  )
+  (gr_text "Grosor de la placa: " (at 91.721423 17.75) (layer "Cmts.User")
+    (effects (font (size 1.5 1.5) (thickness 0.2)) (justify left top))
+  )
+  (gr_text "CARACTERÍSTICAS DE LA PLACA" (at 13 13) (layer "Cmts.User")
+    (effects (font (size 2 2) (thickness 0.4)) (justify left top))
+  )
+  (gr_text "Número de capas de cobre: " (at 13.75 17.75) (layer "Cmts.User")
+    (effects (font (size 1.5 1.5) (thickness 0.2)) (justify left top))
+  )
+  (gr_text "No" (at 129.778565 28.25) (layer "Cmts.User")
+    (effects (font (size 1.5 1.5) (thickness 0.2)) (justify left top))
+  )
+  (gr_text "0,0000 mm / 0,0000 mm" (at 57.664285 24.75) (layer "Cmts.User")
+    (effects (font (size 1.5 1.5) (thickness 0.2)) (justify left top))
+  )
+  (gr_text "2" (at 57.664285 17.75) (layer "Cmts.User")
+    (effects (font (size 1.5 1.5) (thickness 0.2)) (justify left top))
+  )
+  (gr_text "0,3000 mm" (at 129.778565 24.75) (layer "Cmts.User")
+    (effects (font (size 1.5 1.5) (thickness 0.2)) (justify left top))
+  )
+  (gr_text "No" (at 57.664285 35.25) (layer "Cmts.User")
+    (effects (font (size 1.5 1.5) (thickness 0.2)) (justify left top))
+  )
+  (gr_text "No" (at 57.664285 31.75) (layer "Cmts.User")
+    (effects (font (size 1.5 1.5) (thickness 0.2)) (justify left top))
+  )
+  (gr_text "90,0000 mm x 60,0000 mm" (at 57.664285 21.25) (layer "Cmts.User")
+    (effects (font (size 1.5 1.5) (thickness 0.2)) (justify left top))
+  )
+  (gr_text "" (at 91.721423 21.25) (layer "Cmts.User")
+    (effects (font (size 1.5 1.5) (thickness 0.2)) (justify left top))
+  )
+  (gr_text "Conectores laterales de tarjeta: " (at 13.75 35.25) (layer "Cmts.User")
+    (effects (font (size 1.5 1.5) (thickness 0.2)) (justify left top))
+  )
+  (gr_text "None" (at 57.664285 28.25) (layer "Cmts.User")
+    (effects (font (size 1.5 1.5) (thickness 0.2)) (justify left top))
+  )
+  (gr_text "Pads castellados: " (at 13.75 31.75) (layer "Cmts.User")
+    (effects (font (size 1.5 1.5) (thickness 0.2)) (justify left top))
+  )
+  (gr_text "Pista/espaciado mínimo: " (at 13.75 24.75) (layer "Cmts.User")
+    (effects (font (size 1.5 1.5) (thickness 0.2)) (justify left top))
+  )
+  (gr_text "Terminación de cobre: " (at 13.75 28.25) (layer "Cmts.User")
+    (effects (font (size 1.5 1.5) (thickness 0.2)) (justify left top))
+  )
+  (gr_text "Bordes de la placa revestidos: " (at 91.721423 31.75) (layer "Cmts.User")
+    (effects (font (size 1.5 1.5) (thickness 0.2)) (justify left top))
+  )
+  (gr_text "No" (at 129.778565 31.75) (layer "Cmts.User")
+    (effects (font (size 1.5 1.5) (thickness 0.2)) (justify left top))
+  )
+  (gr_text "1,6000 mm" (at 129.778565 17.75) (layer "Cmts.User")
+    (effects (font (size 1.5 1.5) (thickness 0.2)) (justify left top))
+  )
+  (gr_text "Dimensiones generales de la placa: " (at 13.75 21.25) (layer "Cmts.User")
+    (effects (font (size 1.5 1.5) (thickness 0.2)) (justify left top))
+  )
+  (dimension (type aligned) (layer "Cmts.User")
     (pts (xy 196 67) (xy 196 127))
     (height -6)
-    (gr_text "60,0000 mm" (at 200.85 97 90) (layer "Edge.Cuts")
+    (gr_text "60,0000 mm" (at 200.85 97 90) (layer "Cmts.User")
       (effects (font (size 1 1) (thickness 0.15)))
     )
@@
     (style (thickness 0.1) (arrow_length 1.27) (text_position_mode 0) (extension_height 0.58642) (extension_offset 0.5) keep_text_aligned)
   )
-  (dimension (type aligned) (layer "Edge.Cuts")
+  (dimension (type aligned) (layer "Cmts.User")
     (pts (xy 196 67) (xy 106 67))
     (height 3.999999)
-    (gr_text "90,0000 mm" (at 151 61.850001) (layer "Edge.Cuts")
+    (gr_text "90,0000 mm" (at 151 61.850001) (layer "Cmts.User")
       (effects (font (size 1 1) (thickness 0.15)))
     )
@@
     )
   )
+  (group "group-boardCharacteristics" (id cc0fddd3-1024-4935-8204-c01d63e8370a)
+    (members
+      0ad3a937-2de5-47f3-a547-b15f6ec125b9
+      0b65092a-d70c-4aa2-afb1-71cd1bb4d1cf
+      1b704943-6d8e-4b11-99fd-868642619559
+      37b7a786-3d25-4944-8cf0-bb3c848f6d62
+      4afcc0cc-1f1e-4f62-ae9e-8d3a6653dd40
+      56b5be58-125d-4e4f-9b79-186a445d0463
+      56c4d902-2e37-4880-96d5-cdbdbebe00d4
+      5798b8b9-b141-4fc4-b56c-a242179a69a9
+      58963533-30e0-4e21-9d00-7ce59b994041
+      5a707b59-27eb-43ff-b419-40c26b2997a9
+      65dc68f9-df49-41d3-af76-be68c7dc9050
+      6b1a177e-202f-4b19-a793-b060dd1a4fc2
+      74199da0-ef85-42d7-ae4f-5604c8c62291
+      852dcd6e-e71c-4509-a07a-b5437dc9899a
+      99c0490e-538f-4b68-a384-2f35ee1dd4e9
+      b19fd7e2-533b-4be5-98a7-46418369a228
+      b2635ff1-8b71-484f-b5fb-f2a661a2df42
+      b4f0dcf2-a200-4470-8dfd-f2aa750b9f70
+      b78235ba-471f-4d27-ae19-00a8fc0de4f6
+      cb83a04d-92f6-4c0f-8d0b-b8b20bcba9aa
+      d19c5758-17e4-4d9d-b84d-7dce8adf43fb
+      eaea806d-34a9-4d31-bccf-856531eed191
+      fd58c672-5e27-4922-bfab-9a35b0530c1c
+    )
+  )
