File: ngspice_filtro_pasivo.kicad_sch (KiCad schematic)
At the start: 8 parts

Commit message: agregando documentos de fabricacion
Parts:
- C1: value ${SIM.PARAMS} -> 56uF
- H1, H2, H3, H4: now left out of the parts list
- L2: value ${SIM.PARAMS} -> 1.8mH
- R1: value ${SIM.PARAMS} -> 8
Other:
- title: (none) -> Filtro pasa bajas pasivo de segundo orden
